File: eda/BitkanoneV2.sch (KiCad schematic (older format))
At the start: 23 parts, among them J201 5VUSB, J211 Jumper, J212 Jumper, J221 Jumper, J222 Jumper, J231 Jumper, J232 Jumper, J233 Jumper, J234 Jumper, U201 BluePill_STM32F103C, U202 10DOF, U203 MCP2551-I-SN, X101 01x02M, X201 01x03M, X231 Bus, X232 Bus, X233 Bus, X234 Bus, X251 MotorCon

Commit message: WS2812B grid finished
Parts:
- added X990: Conn_01x01, Connector_PinHeader_2.54mm:PinHeader_1x01_P2.54mm_Vertical, symbol Connector_Generic:Conn_01x01
- renumbered C251 to C401, C252 to C402, R202 to R221, R201 to R222, U203 to U202, U202 to U301, X201 to X200, J201 to X201, J211 to X211, J212 to X222, X251 to X401
Connections:
- wire segments 125 -> 127
Changed lines of the file:
@@
 $Descr A4 11693 8268
 encoding utf-8
-Sheet 1 1
+Sheet 1 2
 Title "BitkanoneV2"
 Date "2018-12-08"
@@
 $EndComp
 $Comp
-L power:+5V #PWR0101
+L power:+5V #PWR0909
 U 1 1 5C99DB7A
 P 6000 2850
-F 0 "#PWR0101" H 6000 2700 50  0001 C CNN
+F 0 "#PWR0909" H 6000 2700 50  0001 C CNN
 F 1 "+5V" H 6015 3023 50  0000 C CNN
 F 2 "" H 6000 2850 50  0001 C CNN
@@
 $EndComp
 $Comp
-L power:GND #PWR0102
+L power:GND #PWR0921
 U 1 1 5C99DBA6
 P 3450 5050
-F 0 "#PWR0102" H 3450 4800 50  0001 C CNN
+F 0 "#PWR0921" H 3450 4800 50  0001 C CNN
 F 1 "GND" H 3455 4877 50  0000 C CNN
 F 2 "" H 3450 5050 50  0001 C CNN
@@
 $EndComp
 $Comp
-L power:+3V3 #PWR0103
+L power:+3V3 #PWR0907
 U 1 1 5C99DBF5
 P 5400 2850
-F 0 "#PWR0103" H 5400 2700 50  0001 C CNN
+F 0 "#PWR0907" H 5400 2700 50  0001 C CNN
 F 1 "+3V3" H 5415 3023 50  0000 C CNN
 F 2 "" H 5400 2850 50  0001 C CNN
@@
 $EndComp
 $Comp
-L power:GND #PWR0104
+L power:GND #PWR0908
 U 1 1 5C99DC20
 P 5650 2850
-F 0 "#PWR0104" H 5650 2600 50  0001 C CNN
+F 0 "#PWR0908" H 5650 2600 50  0001 C CNN
 F 1 "GND" H 5655 2677 50  0000 C CNN
 F 2 "" H 5650 2850 50  0001 C CNN
@@
 $EndComp
 $Comp
-L power:+3V3 #PWR0105
+L power:+3V3 #PWR0919
 U 1 1 5C99DC2E
 P 3450 4800
-F 0 "#PWR0105" H 3450 4650 50  0001 C CNN
+F 0 "#PWR0919" H 3450 4650 50  0001 C CNN
 F 1 "+3V3" V 3465 4928 50  0000 L CNN
 F 2 "" H 3450 4800 50  0001 C CNN
@@
 $EndComp
 $Comp
-L Device:Jumper_NC_Small J201
+L Device:Jumper_NC_Small X201
 U 1 1 5C99DCCD
 P 5850 3300
-F 0 "J201" H 5850 3512 50  0000 C CNN
+F 0 "X201" H 5850 3512 50  0000 C CNN
 F 1 "5VUSB" H 5850 3421 50  0000 C CNN
 F 2 "Jumper:SolderJumper-2_P1.3mm_Open_Pad1.0x1.5mm" H 5850 3300 50  0001 C CNN
@@
 $EndComp
 $Comp
-L power:+5V #PWR0106
+L power:+5V #PWR0902
 U 1 1 5C99E955
 P 10000 1500
-F 0 "#PWR0106" H 10000 1350 50  0001 C CNN
+F 0 "#PWR0902" H 10000 1350 50  0001 C CNN
 F 1 "+5V" H 10015 1673 50  0000 C CNN
 F 2 "" H 10000 1500 50  0001 C CNN
@@
 $EndComp
 $Comp
-L power:GND #PWR0107
+L power:GND #PWR0917
 U 1 1 5C99E990
 P 9900 4200
-F 0 "#PWR0107" H 9900 3950 50  0001 C CNN
+F 0 "#PWR0917" H 9900 3950 50  0001 C CNN
 F 1 "GND" H 9905 4027 50  0000 C CNN
 F 2 "" H 9900 4200 50  0001 C CNN
@@
 	5300 4600 5450 4600
 $Comp
-L Device:R R201
+L Device:R R222
 U 1 1 5C9AB29D
 P 8250 2700
-F 0 "R201" H 8320 2746 50  0000 L CNN
+F 0 "R222" H 8320 2746 50  0000 L CNN
 F 1 "1k8" H 8320 2655 50  0000 L CNN
 F 2 "Resistor_SMD:R_0603_1608Metric_Pad1.05x0.95mm_HandSolder" V 8180 2700 50  0001 C CNN
@@
 $EndComp
 $Comp
-L Interface_CAN_LIN:MCP2551-I-SN U203
+L Interface_CAN_LIN:MCP2551-I-SN U202
 U 1 1 5C9ABEC1
 P 7900 1800
-F 0 "U203" H 7900 2378 50  0000 C CNN
+F 0 "U202" H 7900 2378 50  0000 C CNN
 F 1 "MCP2551-I-SN" H 7900 2287 50  0000 C CNN
 F 2 "Package_SO:SOIC-8_3.9x4.9mm_P1.27mm" H 7900 1300 50  0001 C CIN
@@
 	9900 4100 9900 4200
 $Comp
-L power:GND #PWR0108
+L power:GND #PWR0905
 U 1 1 5C9BD061
 P 7900 2300
-F 0 "#PWR0108" H 7900 2050 50  0001 C CNN
+F 0 "#PWR0905" H 7900 2050 50  0001 C CNN
 F 1 "GND" H 7905 2127 50  0000 C CNN
 F 2 "" H 7900 2300 50  0001 C CNN
@@
 $EndComp
 $Comp
-L power:+3V3 #PWR0109
+L power:+3V3 #PWR0901
 U 1 1 5C9BD0A2
 P 7900 1100
-F 0 "#PWR0109" H 7900 950 50  0001 C CNN
+F 0 "#PWR0901" H 7900 950 50  0001 C CNN
 F 1 "+3V3" H 7915 1273 50  0000 C CNN
 F 2 "" H 7900 1100 50  0001 C CNN
@@
 	7900 2200 7900 2250
 $Comp
-L Device:Jumper_NC_Small J211
+L Device:Jumper_NC_Small X211
 U 1 1 5C9C2FE4
 P 8950 1700
-F 0 "J211" H 8950 1912 50  0000 C CNN
+F 0 "X211" H 8950 1912 50  0000 C CNN
 F 1 "Jumper" H 8950 1821 50  0000 C CNN
 F 2 "Jumper:SolderJumper-2_P1.3mm_Open_Pad1.0x1.5mm" H 8950 1700 50  0001 C CNN
@@
 $EndComp
 $Comp
-L Device:Jumper_NC_Small J212
+L Device:Jumper_NC_Small X222
 U 1 1 5C9C4CBB
 P 8950 2000
-F 0 "J212" H 8950 2212 50  0000 C CNN
+F 0 "X222" H 8950 2212 50  0000 C CNN
 F 1 "Jumper" H 8950 2121 50  0000 C CNN
 F 2 "Jumper:SolderJumper-2_P1.3mm_Open_Pad1.0x1.5mm" H 8950 2000 50  0001 C CNN
@@
 $EndComp
 $Comp
-L Device:R R202
+L Device:R R221
 U 1 1 5C9DD3D7
 P 8550 2700
-F 0 "R202" H 8620 2746 50  0000 L CNN
+F 0 "R221" H 8620 2746 50  0000 L CNN
 F 1 "1k8" H 8620 2655 50  0000 L CNN
 F 2 "Resistor_SMD:R_0603_1608Metric_Pad1.05x0.95mm_HandSolder" V 8480 2700 50  0001 C CNN
@@
 	7300 1600 7400 1600
 $Comp
-L power:+3V3 #PWR0110
+L power:+3V3 #PWR0906
 U 1 1 5C9DE51A
 P 8550 2450
-F 0 "#PWR0110" H 8550 2300 50  0001 C CNN
+F 0 "#PWR0906" H 8550 2300 50  0001 C CNN
 F 1 "+3V3" H 8565 2623 50  0000 C CNN
 F 2 "" H 8550 2450 50  0001 C CNN
@@
 Wire Wire Line
 	7900 2250 7900 2300
-Text GLabel 5750 4700 2    50   Input ~ 0
-DIN
-Wire Wire Line
-	5300 4700 5750 4700
 Wire Wire Line
 	5300 4900 5450 4900
@@
 	3450 4600 3550 4600
 $Comp
-L Connector:Conn_01x03_Male X201
+L Connector:Conn_01x03_Male X200
 U 1 1 5CA6E171
 P 6300 4400
-F 0 "X201" H 6273 4330 50  0000 R CNN
+F 0 "X200" H 6273 4330 50  0000 R CNN
 F 1 "01x03M" H 6273 4421 50  0000 R CNN
 F 2 "Connector_PinHeader_2.54mm:PinHeader_1x03_P2.54mm_Vertical" H 6300 4400 50  0001 C CNN
@@
 $EndComp
 $Comp
-L power:GND #PWR0111
+L power:GND #PWR0916
 U 1 1 5CA79F60
 P 6000 4200
-F 0 "#PWR0111" H 6000 3950 50  0001 C CNN
+F 0 "#PWR0916" H 6000 3950 50  0001 C CNN
 F 1 "GND" H 6005 4027 50  0000 C CNN
 F 2 "" H 6000 4200 50  0001 C CNN
@@
 	6000 4300 6100 4300
 $Comp
-L Bitkanone:10DOF U202
+L Bitkanone:10DOF U301
 U 1 1 5CA845C0
 P 1700 2300
-F 0 "U202" H 1927 2351 50  0000 L CNN
+F 0 "U301" H 1927 2351 50  0000 L CNN
 F 1 "10DOF" H 1927 2260 50  0000 L CNN
 F 2 "Connector_PinSocket_2.54mm:PinSocket_1x08_P2.54mm_Vertical" H 1700 2750 50  0001 C CNN
@@
 $EndComp
 $Comp
-L power:GND #PWR0112
+L power:GND #PWR0903
 U 1 1 5CA847D0
 P 1100 1850
-F 0 "#PWR0112" H 1100 1600 50  0001 C CNN
+F 0 "#PWR0903" H 1100 1600 50  0001 C CNN
 F 1 "GND" H 1105 1677 50  0000 C CNN
 F 2 "" H 1100 1850 50  0001 C CNN
@@
 $EndComp
 $Comp
-L power:+3V3 #PWR0113
+L power:+3V3 #PWR0904
 U 1 1 5CA84826
 P 1350 1850
-F 0 "#PWR0113" H 1350 1700 50  0001 C CNN
+F 0 "#PWR0904" H 1350 1700 50  0001 C CNN
 F 1 "+3V3" H 1365 2023 50  0000 C CNN
 F 2 "" H 1350 1850 50  0001 C CNN
@@
 (to Daughterboards)
 $Comp
-L Bitkanone:MotorCon X251
+L Bitkanone:MotorCon X401
 U 1 1 5CAB3F7B
 P 1300 3600
-F 0 "X251" H 1477 3651 50  0000 L CNN
+F 0 "X401" H 1477 3651 50  0000 L CNN
 F 1 "MotorCon" H 1477 3560 50  0000 L CNN
 F 2 "Connector_PinSocket_2.54mm:PinSocket_1x08_P2.54mm_Vertical" H 1200 3850 50  0001 C CNN
@@
 $EndComp
 $Comp
-L power:GND #PWR0114
+L power:GND #PWR0915
 U 1 1 5CAC98DB
 P 2000 3850
-F 0 "#PWR0114" H 2000 3600 50  0001 C CNN
+F 0 "#PWR0915" H 2000 3600 50  0001 C CNN
 F 1 "GND" H 2005 3677 50  0000 C CNN
 F 2 "" H 2000 3850 50  0001 C CNN
@@
 $EndComp
 $Comp
-L power:+5V #PWR0115
+L power:+5V #PWR0912
 U 1 1 5CAC0543
 P 2000 3350
-F 0 "#PWR0115" H 2000 3200 50  0001 C CNN
+F 0 "#PWR0912" H 2000 3200 50  0001 C CNN
 F 1 "+5V" H 2015 3523 50  0000 C CNN
 F 2 "" H 2000 3350 50  0001 C CNN
@@
 $EndComp
 $Comp
-L Device:CP C251
+L Device:CP C401
 U 1 1 5CAE5DA8
 P 2000 3600
-F 0 "C251" H 2118 3646 50  0000 L CNN
+F 0 "C401" H 2118 3646 50  0000 L CNN
 F 1 "220u" H 2118 3555 50  0000 L CNN
 F 2 "Capacitor_SMD:CP_Elec_6.3x5.3" H 2038 3450 50  0001 C CNN
@@
 	2000 3750 2000 3800
 $Comp
-L Device:CP C252
+L Device:CP C402
 U 1 1 5CB1AF06
 P 2450 3600
-F 0 "C252" H 2568 3646 50  0000 L CNN
+F 0 "C402" H 2568 3646 50  0000 L CNN
 F 1 "220u" H 2568 3555 50  0000 L CNN
 F 2 "Capacitor_SMD:CP_Elec_6.3x5.3" H 2488 3450 50  0001 C CNN
@@
 	2000 3400 2000 3450
 $Comp
-L power:GND #PWR0116
+L power:GND #PWR0910
 U 1 1 5CB36D7D
 P 900 3250
-F 0 "#PWR0116" H 900 3000 50  0001 C CNN
+F 0 "#PWR0910" H 900 3000 50  0001 C CNN
 F 1 "GND" V 905 3122 50  0000 R CNN
 F 2 "" H 900 3250 50  0001 C CNN
@@
 $EndComp
 $Comp
-L power:+5V #PWR0117
+L power:+5V #PWR0911
 U 1 1 5CB36DDC
 P 900 3350
-F 0 "#PWR0117" H 900 3200 50  0001 C CNN
+F 0 "#PWR0911" H 900 3200 50  0001 C CNN
 F 1 "+5V" V 915 3478 50  0000 L CNN
 F 2 "" H 900 3350 50  0001 C CNN
@@
 $EndComp
 $Comp
-L power:GND #PWR0118
+L power:GND #PWR0913
 U 1 1 5CB5AA97
 P 900 3650
-F 0 "#PWR0118" H 900 3400 50  0001 C CNN
+F 0 "#PWR0913" H 900 3400 50  0001 C CNN
 F 1 "GND" V 905 3522 50  0000 R CNN
 F 2 "" H 900 3650 50  0001 C CNN
@@
 $EndComp
 $Comp
-L power:+5V #PWR0119
+L power:+5V #PWR0914
 U 1 1 5CB5AA9D
 P 900 3750
-F 0 "#PWR0119" H 900 3600 50  0001 C CNN
+F 0 "#PWR0914" H 900 3600 50  0001 C CNN
 F 1 "+5V" V 915 3878 50  0000 L CNN
 F 2 "" H 900 3750 50  0001 C CNN
@@
 $EndComp
 $Comp
-L power:+5V #PWR0120
+L power:+5V #PWR0918
 U 1 1 5CB9ED1E
 P 1800 4600
-F 0 "#PWR0120" H 1800 4450 50  0001 C CNN
+F 0 "#PWR0918" H 1800 4450 50  0001 C CNN
 F 1 "+5V" H 1815 4773 50  0000 C CNN
 F 2 "" H 1800 4600 50  0001 C CNN
@@
 $EndComp
 $Comp
-L power:GND #PWR0121
+L power:GND #PWR0920
 U 1 1 5CB9EE6B
 P 1800 4900
-F 0 "#PWR0121" H 1800 4650 50  0001 C CNN
+F 0 "#PWR0920" H 1800 4650 50  0001 C CNN
 F 1 "GND" H 1805 4727 50  0000 C CNN
 F 2 "" H 1800 4900 50  0001 C CNN
@@
 Text Notes 10800 1700 0    50   ~ 0
 Top
+$Sheet
+S 3950 6700 1600 700
+U 5C0C4423
+F0 "LedGrid" 50
+F1 "LedGrid.sch" 50
+F2 "DIN" I L 3950 6800 50
+F3 "DOUT" O R 5550 6800 50
+$EndSheet
+Text Label 5450 4700 0    50   ~ 0
+DIN
+Text Label 3850 6800 2    50   ~ 0
+DIN
+Wire Wire Line
+	3850 6800 3950 6800
+Wire Wire Line
+	5300 4700 5450 4700
+Wire Wire Line
+	5550 6800 5650 6800
+$Comp
+L Connector_Generic:Conn_01x01 X990
+U 1 1 5C1992BC
+P 5850 6800
+F 0 "X990" H 5930 6842 50  0000 L CNN
+F 1 "Conn_01x01" H 5930 6751 50  0000 L CNN
+F 2 "Connector_PinHeader_2.54mm:PinHeader_1x01_P2.54mm_Vertical" H 5850 6800 50  0001 C CNN
+F 3 "~" H 5850 6800 50  0001 C CNN
+	1    5850 6800
+	1    0    0    -1
+$EndComp
 $EndSCHEMATC

Commit message: placement finished
Parts:
- removed J221, J222: Jumper, Jumper:SolderJumper-2_P1.3mm_Open_Pad1.0x1.5mm, symbol Device:Jumper_NO_Small
- removed X211, X222: Jumper, Jumper:SolderJumper-2_P1.3mm_Open_Pad1.0x1.5mm, symbol Device:Jumper_NC_Small
- added J211: JH23, Jumper:SolderJumper-3_P1.3mm_Open_RoundedPad1.0x1.5mm_NumberLabels, symbol Jumper:SolderJumper_3_Open
- added J212: JL23, Jumper:SolderJumper-3_P1.3mm_Open_RoundedPad1.0x1.5mm_NumberLabels, symbol Jumper:SolderJumper_3_Open
- U201: footprint BluePill_breakouts:BluePill_STM32F103C -> BluePill_breakouts:BluePill_STM32F103C_Center_NoPROG; symbol bluepill_breakouts:BluePill_STM32F103C -> bluepill_breakouts:BluePill_STM32F103C_NoProg
Connections:
- wire segments 127 -> 126
Changed lines of the file:
@@
 $EndDescr
 $Comp
-L bluepill_breakouts:BluePill_STM32F103C U201
+L bluepill_breakouts:BluePill_STM32F103C_NoProg U201
 U 1 1 5C99DAC3
 P 4400 3800
 F 0 "U201" H 4425 2328 50  0000 C CNN
 F 1 "BluePill_STM32F103C" H 4425 2237 50  0000 C CNN
-F 2 "BluePill_breakouts:BluePill_STM32F103C" H 4450 2200 50  0001 C CNN
+F 2 "BluePill_breakouts:BluePill_STM32F103C_Center_NoPROG" H 4450 2200 50  0001 C CNN
 F 3 "www.rogerclark.net" H 4400 2300 50  0001 C CNN
 	1    4400 3800
@@
 	7900 2200 7900 2250
 $Comp
-L Device:Jumper_NC_Small X211
-U 1 1 5C9C2FE4
-P 8950 1700
-F 0 "X211" H 8950 1912 50  0000 C CNN
-F 1 "Jumper" H 8950 1821 50  0000 C CNN
-F 2 "Jumper:SolderJumper-2_P1.3mm_Open_Pad1.0x1.5mm" H 8950 1700 50  0001 C CNN
-F 3 "~" H 8950 1700 50  0001 C CNN
-	1    8950 1700
-	1    0    0    -1
-$EndComp
-$Comp
-L Device:Jumper_NC_Small X222
-U 1 1 5C9C4CBB
-P 8950 2000
-F 0 "X222" H 8950 2212 50  0000 C CNN
-F 1 "Jumper" H 8950 2121 50  0000 C CNN
-F 2 "Jumper:SolderJumper-2_P1.3mm_Open_Pad1.0x1.5mm" H 8950 2000 50  0001 C CNN
-F 3 "~" H 8950 2000 50  0001 C CNN
-	1    8950 2000
-	1    0    0    -1
-$EndComp
-$Comp
-L Device:Jumper_NO_Small J221
-U 1 1 5C9D0165
-P 9100 2900
-F 0 "J221" H 9100 3085 50  0000 C CNN
-F 1 "Jumper" H 9100 2994 50  0000 C CNN
-F 2 "Jumper:SolderJumper-2_P1.3mm_Open_Pad1.0x1.5mm" H 9100 2900 50  0001 C CNN
-F 3 "~" H 9100 2900 50  0001 C CNN
-	1    9100 2900
-	1    0    0    -1
-$EndComp
-$Comp
-L Device:Jumper_NO_Small J222
-U 1 1 5C9D01D2
-P 8800 3050
-F 0 "J222" H 8800 3235 50  0000 C CNN
-F 1 "Jumper" H 8800 3144 50  0000 C CNN
-F 2 "Jumper:SolderJumper-2_P1.3mm_Open_Pad1.0x1.5mm" H 8800 3050 50  0001 C CNN
-F 3 "~" H 8800 3050 50  0001 C CNN
-	1    8800 3050
-	1    0    0    -1
-$EndComp
-$Comp
 L Device:R R221
 U 1 1 5C9DD3D7
@@
 	8550 2850 8550 2900
 Wire Wire Line
-	8550 2900 9000 2900
-Wire Wire Line
-	8250 3050 8700 3050
-Wire Wire Line
 	6900 1600 7300 1600
 Connection ~ 7300 1600
@@
 Wire Wire Line
 	5400 3500 5300 3500
-Text Notes 8750 2600 0    50   ~ 0
+Text Notes 8150 2400 0    50   ~ 0
 I2C-Bus
 Wire Wire Line
 	7200 3050 8250 3050
-Connection ~ 8250 3050
 Wire Wire Line
 	8250 2850 8250 3050
@@
 Wire Wire Line
 	7300 2900 8550 2900
-Connection ~ 8550 2900
 Wire Notes Line
 	8100 2200 9250 2200
@@
 	10350 1700 9800 1700
 Wire Wire Line
-	9800 1700 9800 2400
-Wire Wire Line
 	10350 3100 9800 3100
 Connection ~ 9800 3100
@@
 Connection ~ 9800 2400
 Wire Wire Line
-	9800 2400 9800 2900
-Wire Wire Line
 	10350 1800 9700 1800
 Wire Wire Line
-	9700 1800 9700 2000
-Wire Wire Line
 	9700 2500 10350 2500
 Wire Wire Line
 	10350 3200 9700 3200
-Wire Wire Line
-	9700 3200 9700 3050
 Connection ~ 9700 2500
 Wire Wire Line
 	9700 3900 9700 3200
 Connection ~ 9700 3200
-Wire Wire Line
-	9200 2900 9800 2900
-Connection ~ 9800 2900
-Wire Wire Line
-	9800 2900 9800 3100
-Wire Wire Line
-	8900 3050 9700 3050
-Connection ~ 9700 3050
-Wire Wire Line
-	9700 3050 9700 2500
-Wire Wire Line
-	9050 1700 9800 1700
-Connection ~ 9800 1700
-Wire Wire Line
-	9050 2000 9700 2000
-Connection ~ 9700 2000
-Wire Wire Line
-	9700 2000 9700 2500
-Wire Wire Line
-	8850 1700 8400 1700
-Wire Wire Line
-	8400 1900 8550 1900
-Wire Wire Line
-	8550 1900 8550 2000
-Wire Wire Line
-	8550 2000 8850 2000
 Wire Notes Line
 	2900 900  2900 5600
@@
 	1    0    0    -1
 $EndComp
+$Comp
+L Jumper:SolderJumper_3_Open J211
+U 1 1 5C0D4078
+P 9200 2000
+F 0 "J211" V 9246 2068 50  0000 L CNN
+F 1 "JH23" V 9155 2068 50  0000 L CNN
+F 2 "Jumper:SolderJumper-3_P1.3mm_Open_RoundedPad1.0x1.5mm_NumberLabels" H 9200 2000 50  0001 C CNN
+F 3 "~" H 9200 2000 50  0001 C CNN
+	1    9200 2000
+	0    -1   -1   0
+$EndComp
+Wire Wire Line
+	9700 2500 9700 3200
+Wire Wire Line
+	9800 2400 9800 3100
+$Comp
+L Jumper:SolderJumper_3_Open J212
+U 1 1 5C0E0693
+P 8900 2400
+F 0 "J212" V 8946 2468 50  0000 L CNN
+F 1 "JL23" V 8855 2468 50  0000 L CNN
+F 2 "Jumper:SolderJumper-3_P1.3mm_Open_RoundedPad1.0x1.5mm_NumberLabels" H 8900 2400 50  0001 C CNN
+F 3 "~" H 8900 2400 50  0001 C CNN
+	1    8900 2400
+	0    -1   -1   0
+$EndComp
+Wire Wire Line
+	8250 3050 8900 3050
+Wire Wire Line
+	8900 3050 8900 2600
+Connection ~ 8250 3050
+Connection ~ 8550 2900
+Wire Wire Line
+	9050 2400 9700 2400
+Connection ~ 9700 2400
+Wire Wire Line
+	9700 2400 9700 2500
+Wire Wire Line
+	9700 1800 9700 2400
+Wire Wire Line
+	8400 1900 8900 1900
+Wire Wire Line
+	8900 1900 8900 2200
+Wire Wire Line
+	9800 1700 9800 2000
+Wire Wire Line
+	9200 2900 9200 2200
+Wire Wire Line
+	8550 2900 9200 2900
+Wire Wire Line
+	9350 2000 9800 2000
+Connection ~ 9800 2000
+Wire Wire Line
+	9800 2000 9800 2400
+Wire Wire Line
+	9200 1700 9200 1800
+Wire Wire Line
+	8400 1700 9200 1700
 $EndSCHEMATC

Commit message: all but bus routed
Connections:
- net labels added: CANH, CANL
Changed lines of the file:
@@
 L power:+5V #PWR0918
 U 1 1 5CB9ED1E
+P 1800 4900
+F 0 "#PWR0918" H 1800 4750 50  0001 C CNN
+F 1 "+5V" H 1815 5073 50  0000 C CNN
+F 2 "" H 1800 4900 50  0001 C CNN
+F 3 "" H 1800 4900 50  0001 C CNN
+	1    1800 4900
+	-1   0    0    1
+$EndComp
+$Comp
+L power:GND #PWR0920
+U 1 1 5CB9EE6B
 P 1800 4600
-F 0 "#PWR0918" H 1800 4450 50  0001 C CNN
-F 1 "+5V" H 1815 4773 50  0000 C CNN
+F 0 "#PWR0920" H 1800 4350 50  0001 C CNN
+F 1 "GND" H 1805 4427 50  0000 C CNN
 F 2 "" H 1800 4600 50  0001 C CNN
 F 3 "" H 1800 4600 50  0001 C CNN
 	1    1800 4600
-	1    0    0    -1
-$EndComp
-$Comp
-L power:GND #PWR0920
-U 1 1 5CB9EE6B
-P 1800 4900
-F 0 "#PWR0920" H 1800 4650 50  0001 C CNN
-F 1 "GND" H 1805 4727 50  0000 C CNN
-F 2 "" H 1800 4900 50  0001 C CNN
-F 3 "" H 1800 4900 50  0001 C CNN
-	1    1800 4900
-	1    0    0    -1
-$EndComp
-Wire Wire Line
-	1700 4800 1800 4800
+	-1   0    0    1
+$EndComp
 Wire Wire Line
 	1800 4800 1800 4900
-Wire Wire Line
-	1700 4700 1800 4700
 Wire Wire Line
 	1800 4700 1800 4600
@@
 Wire Wire Line
 	8400 1700 9200 1700
+Wire Wire Line
+	1700 4700 1800 4700
+Wire Wire Line
+	1800 4800 1700 4800
+Text Label 9350 2000 0    50   ~ 0
+CANH
+Text Label 9350 2400 0    50   ~ 0
+CANL
 $EndSCHEMATC

Commit message: routing finished
Parts:
- added X990: Conn_01x01, Connector_PinHeader_2.54mm:PinHeader_1x01_P2.54mm_Vertical, symbol Connector_Generic:Conn_01x01
- renumbered X990 to X991
Changed lines of the file:
@@
 Text Label 9350 3300 0    50   ~ 0
 TBottom
-Text Label 5450 4900 0    50   ~ 0
+Text Label 5450 4100 0    50   ~ 0
 TTop
+Text Label 3450 4000 2    50   ~ 0
+TRight
 Text Label 5450 5000 0    50   ~ 0
-TRight
-Text Label 5450 4800 0    50   ~ 0
 TLeft
-Text Label 5450 4600 0    50   ~ 0
+Text Label 3450 4200 2    50   ~ 0
 TBottom
 Wire Wire Line
 	5300 5000 5450 5000
-Wire Wire Line
-	5300 4800 5450 4800
-Wire Wire Line
-	5300 4600 5450 4600
 $Comp
 L Device:R R222
@@
 	7900 2250 7900 2300
 Wire Wire Line
-	5300 4900 5450 4900
+	5300 4100 5450 4100
 Text Notes 9000 1200 2    118  ~ 24
 Bus
@@
 DIN
 Wire Wire Line
-	3850 6800 3950 6800
-Wire Wire Line
 	5300 4700 5450 4700
 Wire Wire Line
 	5550 6800 5650 6800
 $Comp
-L Connector_Generic:Conn_01x01 X990
+L Connector_Generic:Conn_01x01 X991
 U 1 1 5C1992BC
 P 5850 6800
-F 0 "X990" H 5930 6842 50  0000 L CNN
+F 0 "X991" H 5930 6842 50  0000 L CNN
 F 1 "Conn_01x01" H 5930 6751 50  0000 L CNN
 F 2 "Connector_PinHeader_2.54mm:PinHeader_1x01_P2.54mm_Vertical" H 5850 6800 50  0001 C CNN
@@
 Text Label 9350 2400 0    50   ~ 0
 CANL
+$Comp
+L Connector_Generic:Conn_01x01 X990
+U 1 1 5C129EF7
+P 3450 6800
+F 0 "X990" H 3530 6842 50  0000 L CNN
+F 1 "Conn_01x01" H 3530 6751 50  0000 L CNN
+F 2 "Connector_PinHeader_2.54mm:PinHeader_1x01_P2.54mm_Vertical" H 3450 6800 50  0001 C CNN
+F 3 "~" H 3450 6800 50  0001 C CNN
+	1    3450 6800
+	-1   0    0    1
+$EndComp
+Wire Wire Line
+	3650 6800 3950 6800
+Wire Wire Line
+	3450 4000 3550 4000
+Wire Wire Line
+	3450 4200 3550 4200
 $EndSCHEMATC

Commit message: U301:more space; Phototransistors, Buttons and X42 added
Parts:
- added Q501, Q502: PH_NPN, LED_THT:LED_D3.0mm, symbol Device:Q_Photo_NPN
- added R501, R502: 1k8, Resistor_SMD:R_0603_1608Metric_Pad1.05x0.95mm_HandSolder, symbol Device:R
- added S1, S2, S3: SW, Button_Switch_SMD:SW_SPST_FSMSM, symbol Switch:SW_Push
- added X102: 01x02M, Connector_PinHeader_2.54mm:PinHeader_1x02_P2.54mm_Vertical, symbol Connector:Conn_01x02_Male
- added X42: Conn_01x07_Male, Connector_PinSocket_2.54mm:PinSocket_1x08_P2.54mm_Vertical, symbol Connector:Conn_01x08_Male
- U301: value 10DOF -> 6DOF; symbol Bitkanone:10DOF -> Bitkanone:6DOF
Connections:
- net labels added: Photo1, Photo2, X42_PB3, X42_PB4, X42_PB5, X42_SCL, X42_SDA
- wire segments 126 -> 172
Other:
- note added: "Sensors"
- moved on the sheet: C401, C402, U201, X101, X201, X401

Commit message: silk screen documentation added
Parts:
- added J202: 5VUSB, Connector_PinSocket_2.54mm:PinSocket_1x02_P2.54mm_Vertical, symbol Device:Jumper_NC_Small
- X201: symbol Device:Jumper_NC_Small -> Jumper:SolderJumper_2_Open
Connections:
- net +5V: now also J202.2
- net TX1: now reaches U201.26 (PA9_TX1), X200.1 (Pin_1)
- net RX1: now reaches U201.27 (PA10_RX1), X200.2 (Pin_2)
- net at U201.38 (5V_USB), X201.1 (A): now also J202.1
Changed lines of the file:
@@
 L power:+5V #PWR0909
 U 1 1 5C99DB7A
-P 6300 2850
-F 0 "#PWR0909" H 6300 2700 50  0001 C CNN
-F 1 "+5V" H 6315 3023 50  0000 C CNN
-F 2 "" H 6300 2850 50  0001 C CNN
-F 3 "" H 6300 2850 50  0001 C CNN
-	1    6300 2850
+P 6450 2850
+F 0 "#PWR0909" H 6450 2700 50  0001 C CNN
+F 1 "+5V" H 6465 3023 50  0000 C CNN
+F 2 "" H 6450 2850 50  0001 C CNN
+F 3 "" H 6450 2850 50  0001 C CNN
+	1    6450 2850
 	1    0    0    -1
 $EndComp
@@
 $EndComp
 $Comp
-L Device:Jumper_NC_Small X201
+L Jumper:SolderJumper_2_Open X201
 U 1 1 5C99DCCD
-P 6150 3300
-F 0 "X201" H 6150 3512 50  0000 C CNN
-F 1 "5VUSB" H 6150 3421 50  0000 C CNN
-F 2 "Jumper:SolderJumper-2_P1.3mm_Open_Pad1.0x1.5mm" H 6150 3300 50  0001 C CNN
-F 3 "~" H 6150 3300 50  0001 C CNN
-	1    6150 3300
+P 6250 3000
+F 0 "X201" H 6250 3212 50  0000 C CNN
+F 1 "5VUSB" H 6250 3121 50  0000 C CNN
+F 2 "Jumper:SolderJumper-2_P1.3mm_Open_Pad1.0x1.5mm" H 6250 3000 50  0001 C CNN
+F 3 "~" H 6250 3000 50  0001 C CNN
+	1    6250 3000
 	1    0    0    -1
 $EndComp
@@
 	5950 3200 5950 2850
 Wire Wire Line
-	6250 3300 6300 3300
-Wire Wire Line
-	6300 3300 6300 2850
+	6450 3300 6450 3000
 Wire Wire Line
 	3850 5000 3750 5000
@@
 Text Label 5750 3500 0    50   ~ 0
 CANRX
-Wire Wire Line
-	5600 3300 6050 3300
 Text Notes 8150 2400 0    50   ~ 0
 I2C-Bus
@@
 Wire Wire Line
 	1350 6200 1450 6200
+$Comp
+L Device:Jumper_NC_Small J202
+U 1 1 5C1073B3
+P 6250 3300
+F 0 "J202" H 6250 3512 50  0000 C CNN
+F 1 "5VUSB" H 6250 3421 50  0000 C CNN
+F 2 "Connector_PinSocket_2.54mm:PinSocket_1x02_P2.54mm_Vertical" H 6250 3300 50  0001 C CNN
+F 3 "~" H 6250 3300 50  0001 C CNN
+	1    6250 3300
+	1    0    0    -1
+$EndComp
+Wire Wire Line
+	6350 3300 6450 3300
+Wire Wire Line
+	5600 3300 6050 3300
+Wire Wire Line
+	6100 3000 6050 3000
+Wire Wire Line
+	6050 3000 6050 3300
+Connection ~ 6050 3300
+Wire Wire Line
+	6050 3300 6150 3300
+Wire Wire Line
+	6400 3000 6450 3000
+Connection ~ 6450 3000
+Wire Wire Line
+	6450 3000 6450 2850
+Text Label 5750 4500 0    50   ~ 0
+TX1
+Text Label 5750 4400 0    50   ~ 0
+RX1
 $EndSCHEMATC
