File: eda/BitkanoneV2.sch (KiCad schematic (older format))
At the start: 48 parts, among them J202 5VUSB, J211 JH23, J212 JL23, J231 Jumper, J232 Jumper, J233 Jumper, J234 Jumper, Q501 PH_NPN, Q502 PH_NPN, U201 BluePill_STM32F103C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

Commit message: schematic: ledcom cathode fixed
Connections:
- net GND: no longer R831.2, R832.2, R833.2, R834.2
- new net LedCom: R831.2, R832.2, R833.2, R834.2
Other:
- note added: "Idee Matthias: Ledcom Magnet über TOPO pins\nLeitungen durch Groundguards"
- note removed: "Idee Matthias: Ledcom Magnet über TOPO pins"
Changed lines of the file:
@@
 $EndComp
 Text Notes 6900 3300 0    50   ~ 0
-Idee Matthias: Ledcom Magnet über TOPO pins
-$Comp
-L power:GND #PWR?
-U 1 1 5C2A7DE0
-P 7050 4500
-F 0 "#PWR?" H 7050 4250 50  0001 C CNN
-F 1 "GND" H 7055 4327 50  0000 C CNN
-F 2 "" H 7050 4500 50  0001 C CNN
-F 3 "" H 7050 4500 50  0001 C CNN
-	1    7050 4500
-	1    0    0    -1
-$EndComp
+Idee Matthias: Ledcom Magnet über TOPO pins\nLeitungen durch Groundguards
 Wire Wire Line
 	7050 4000 7050 4100
@@
 F 3 "~" H 7400 4250 50  0001 C CNN
 	1    7400 4250
-	1    0    0    -1
-$EndComp
-$Comp
-L power:GND #PWR?
-U 1 1 5C2FCD25
-P 7400 4500
-F 0 "#PWR?" H 7400 4250 50  0001 C CNN
-F 1 "GND" H 7405 4327 50  0000 C CNN
-F 2 "" H 7400 4500 50  0001 C CNN
-F 3 "" H 7400 4500 50  0001 C CNN
-	1    7400 4500
 	1    0    0    -1
 $EndComp
@@
 	1    0    0    -1
 $EndComp
-$Comp
-L power:GND #PWR?
-U 1 1 5C309193
-P 7750 4500
-F 0 "#PWR?" H 7750 4250 50  0001 C CNN
-F 1 "GND" H 7755 4327 50  0000 C CNN
-F 2 "" H 7750 4500 50  0001 C CNN
-F 3 "" H 7750 4500 50  0001 C CNN
-	1    7750 4500
-	1    0    0    -1
-$EndComp
 Wire Wire Line
 	7750 4000 7750 4100
@@
 	1    0    0    -1
 $EndComp
-$Comp
-L power:GND #PWR?
-U 1 1 5C315A67
-P 8100 4500
-F 0 "#PWR?" H 8100 4250 50  0001 C CNN
-F 1 "GND" H 8105 4327 50  0000 C CNN
-F 2 "" H 8100 4500 50  0001 C CNN
-F 3 "" H 8100 4500 50  0001 C CNN
-	1    8100 4500
-	1    0    0    -1
-$EndComp
 Wire Wire Line
 	8100 4000 8100 4100
@@
 Wire Wire Line
 	8100 3700 8100 3600
+Wire Wire Line
+	8100 4500 7750 4500
+Wire Wire Line
+	7400 4500 7050 4500
+Connection ~ 7400 4500
+Wire Wire Line
+	7400 4500 7750 4500
+Connection ~ 7750 4500
+Text Label 7050 4900 1    50   ~ 0
+LedCom
+Wire Wire Line
+	7050 4500 7050 4900
+Connection ~ 7050 4500
 $EndSCHEMATC
